File: marklin-wifi-ctrl/power_supply.kicad_sch (KiCad schematic)
At the start: 8 parts, among them U300 XL1509-3.3E1

Commit message: Rewrite power supply to use direct wires instead of net labels
Replace scattered net labels (VIN, VSW, +3V3) with direct wire
connections between components, matching the style of all other
generator scripts. Also documents the KiCad wiring rule that wire
segments must terminate at pin locations.

Co-Authored-By: Claude Opus 4.6 <noreply@anthropic.com>
Connections:
- net VIN: no longer names the net of C300.1, C301.1, D300.3 (+), U300.1 (VIN), U300.4 (~{EN})
- net VSW: no longer names the net of D301.1 (K), L300.1, U300.2 (OUT)
Changed lines of the file:
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@@
 		)
-	)
-	(wire
-		(pts (xy 62.23 74.93) (xy 69.85 74.93))
-		(stroke (width 0) (type solid))
-	)
-	(label "VIN"
-		(at 69.85 74.93 0)
-		(fields_autoplaced yes)
-		(effects (font (size 1.27 1.27)) (justify left bottom))
 	)
 	(symbol
@@
 	)
 	(wire
-		(pts (xy 74.93 71.12) (xy 82.55 71.12))
-		(stroke (width 0) (type solid))
-	)
-	(label "VIN"
-		(at 74.93 71.12 180)
-		(fields_autoplaced yes)
-		(effects (font (size 1.27 1.27)) (justify right bottom))
-	)
-	(wire
 		(pts (xy 82.55 78.74) (xy 82.55 86.36))
 		(stroke (width 0) (type solid))
@@
 			)
 		)
-	)
-	(wire
-		(pts (xy 88.9 71.12) (xy 96.52 71.12))
-		(stroke (width 0) (type solid))
-	)
-	(label "VIN"
-		(at 88.9 71.12 180)
-		(fields_autoplaced yes)
-		(effects (font (size 1.27 1.27)) (justify right bottom))
 	)
 	(wire
@@
 	)
 	(wire
-		(pts (xy 111.76 67.31) (xy 119.38 67.31))
-		(stroke (width 0) (type solid))
-	)
-	(label "VIN"
-		(at 111.76 67.31 180)
-		(fields_autoplaced yes)
-		(effects (font (size 1.27 1.27)) (justify right bottom))
-	)
-	(wire
-		(pts (xy 111.76 72.39) (xy 119.38 72.39))
-		(stroke (width 0) (type solid))
-	)
-	(label "VIN"
-		(at 111.76 72.39 180)
-		(fields_autoplaced yes)
-		(effects (font (size 1.27 1.27)) (justify right bottom))
-	)
-	(wire
 		(pts (xy 129.54 77.47) (xy 129.54 85.09))
 		(stroke (width 0) (type solid))
@@
 	)
 	(wire
-		(pts (xy 139.7 67.31) (xy 147.32 67.31))
-		(stroke (width 0) (type solid))
-	)
-	(label "VSW"
-		(at 147.32 67.31 0)
-		(fields_autoplaced yes)
-		(effects (font (size 1.27 1.27)) (justify left bottom))
-	)
-	(wire
-		(pts (xy 139.7 72.39) (xy 147.32 72.39))
-		(stroke (width 0) (type solid))
-	)
-	(label "+3V3"
-		(at 147.32 72.39 0)
-		(fields_autoplaced yes)
-		(effects (font (size 1.27 1.27)) (justify left bottom))
+		(pts (xy 62.23 74.93) (xy 62.23 71.12))
+		(stroke (width 0) (type solid))
+	)
+	(wire
+		(pts (xy 62.23 71.12) (xy 82.55 71.12))
+		(stroke (width 0) (type solid))
+	)
+	(wire
+		(pts (xy 82.55 71.12) (xy 96.52 71.12))
+		(stroke (width 0) (type solid))
+	)
+	(wire
+		(pts (xy 96.52 71.12) (xy 119.38 71.12))
+		(stroke (width 0) (type solid))
+	)
+	(wire
+		(pts (xy 119.38 71.12) (xy 119.38 67.31))
+		(stroke (width 0) (type solid))
+	)
+	(wire
+		(pts (xy 119.38 71.12) (xy 119.38 72.39))
+		(stroke (width 0) (type solid))
+	)
+	(junction
+		(at 82.55 71.12)
+		(diameter 0)
+		(color 0 0 0 0)
+	)
+	(junction
+		(at 96.52 71.12)
+		(diameter 0)
+		(color 0 0 0 0)
+	)
+	(junction
+		(at 119.38 71.12)
+		(diameter 0)
+		(color 0 0 0 0)
 	)
 	(symbol
@@
 	)
 	(wire
-		(pts (xy 147.32 73.66) (xy 154.94 73.66))
-		(stroke (width 0) (type solid))
-	)
-	(label "VSW"
-		(at 147.32 73.66 180)
-		(fields_autoplaced yes)
-		(effects (font (size 1.27 1.27)) (justify right bottom))
-	)
-	(wire
 		(pts (xy 154.94 81.28) (xy 154.94 88.9))
 		(stroke (width 0) (type solid))
@@
 	)
 	(wire
-		(pts (xy 158.75 67.31) (xy 166.37 67.31))
-		(stroke (width 0) (type solid))
-	)
-	(label "VSW"
-		(at 158.75 67.31 180)
-		(fields_autoplaced yes)
-		(effects (font (size 1.27 1.27)) (justify right bottom))
-	)
-	(wire
-		(pts (xy 173.99 67.31) (xy 181.61 67.31))
-		(stroke (width 0) (type solid))
-	)
-	(label "+3V3"
-		(at 181.61 67.31 0)
-		(fields_autoplaced yes)
-		(effects (font (size 1.27 1.27)) (justify left bottom))
+		(pts (xy 139.7 67.31) (xy 154.94 67.31))
+		(stroke (width 0) (type solid))
+	)
+	(wire
+		(pts (xy 154.94 67.31) (xy 166.37 67.31))
+		(stroke (width 0) (type solid))
+	)
+	(wire
+		(pts (xy 154.94 67.31) (xy 154.94 73.66))
+		(stroke (width 0) (type solid))
+	)
+	(junction
+		(at 154.94 67.31)
+		(diameter 0)
+		(color 0 0 0 0)
 	)
 	(symbol
@@
 	)
 	(wire
-		(pts (xy 184.15 71.12) (xy 191.77 71.12))
-		(stroke (width 0) (type solid))
-	)
-	(label "+3V3"
-		(at 184.15 71.12 180)
-		(fields_autoplaced yes)
-		(effects (font (size 1.27 1.27)) (justify right bottom))
-	)
-	(wire
 		(pts (xy 191.77 78.74) (xy 191.77 86.36))
 		(stroke (width 0) (type solid))
@@
 	)
 	(wire
-		(pts (xy 199.39 71.12) (xy 207.01 71.12))
-		(stroke (width 0) (type solid))
-	)
-	(label "+3V3"
-		(at 199.39 71.12 180)
-		(fields_autoplaced yes)
-		(effects (font (size 1.27 1.27)) (justify right bottom))
-	)
-	(wire
 		(pts (xy 207.01 78.74) (xy 207.01 86.36))
 		(stroke (width 0) (type solid))
@@
 	)
 	(wire
+		(pts (xy 173.99 67.31) (xy 173.99 71.12))
+		(stroke (width 0) (type solid))
+	)
+	(wire
+		(pts (xy 173.99 71.12) (xy 191.77 71.12))
+		(stroke (width 0) (type solid))
+	)
+	(wire
+		(pts (xy 191.77 71.12) (xy 207.01 71.12))
+		(stroke (width 0) (type solid))
+	)
+	(wire
+		(pts (xy 139.7 72.39) (xy 173.99 72.39))
+		(stroke (width 0) (type solid))
+	)
+	(wire
+		(pts (xy 173.99 72.39) (xy 173.99 71.12))
+		(stroke (width 0) (type solid))
+	)
+	(junction
+		(at 173.99 71.12)
+		(diameter 0)
+		(color 0 0 0 0)
+	)
+	(wire
